File: shield/GBAHD_Shield.sch (KiCad schematic (older format))
At the start: 38 parts, among them J1 Conn_01x01, J10 Conn_01x10, J11 Conn_02x03_Odd_Even, J12 Conn_01x01, J2 FFC_OGBA_32, J3 FFC_GBA-SP, J4 Conn_01x16, J5 FFC_OGBA_40, J6 Conn_01x06, J7 Conn_01x08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

Commit message: Switched Voltage Regulator to SOT-223 package and Push Button to THT
Parts:
- SW1: footprint Button_Switch_SMD:SW_Push_1P1T_NO_CK_KMR2 -> Button_Switch_THT:SW_PUSH_6mm
- U1: value AZ1117R-ADJ -> AMS1117-ADJ; footprint Package_TO_SOT_SMD:SOT-89-3 -> Package_TO_SOT_SMD:SOT-223-3_TabPin2; symbol Regulator_Linear:AZ1117R-ADJ -> Regulator_Linear:AMS1117
Other:
- moved on the sheet: C2, R2
Changed lines of the file:
@@
 Comment1 "Idea by: sanchezand"
 Comment2 "made by: ManCloud"
-Comment3 "Version: v20210406"
-Comment4 ""
+Comment3 "modified by: hagi"
+Comment4 "Version: v20210406_1"
 $EndDescr
 $Comp
@@
 L Device:C C2
 U 1 1 609BF4FF
-P 1700 4100
-F 0 "C2" H 1800 4000 50  0000 C CNN
-F 1 "22u" H 1600 4200 50  0000 C CNN
-F 2 "Capacitor_SMD:C_0805_2012Metric_Pad1.18x1.45mm_HandSolder" H 1738 3950 50  0001 C CNN
-F 3 "~" H 1700 4100 50  0001 C CNN
-	1    1700 4100
+P 1750 4100
+F 0 "C2" H 1675 4000 50  0000 C CNN
+F 1 "22u" H 1650 4200 50  0000 C CNN
+F 2 "Capacitor_SMD:C_0805_2012Metric_Pad1.18x1.45mm_HandSolder" H 1788 3950 50  0001 C CNN
+F 3 "~" H 1750 4100 50  0001 C CNN
+	1    1750 4100
 	-1   0    0    1
 $EndComp
 Wire Wire Line
-	1700 3850 1700 3900
-Connection ~ 1700 3900
-Wire Wire Line
-	1700 3900 1700 3950
-Wire Wire Line
-	1700 4250 1700 4300
+	1750 3850 1750 3900
+Connection ~ 1750 3900
+Wire Wire Line
+	1750 3900 1750 3950
+Wire Wire Line
+	1750 4250 1750 4300
 Wire Notes Line
 	550  3500 550  7750
@@
 L power:GND #PWR09
 U 1 1 610E1DA2
-P 1700 4300
-F 0 "#PWR09" H 1700 4050 50  0001 C CNN
-F 1 "GND" H 1705 4127 50  0000 C CNN
-F 2 "" H 1700 4300 50  0001 C CNN
-F 3 "" H 1700 4300 50  0001 C CNN
-	1    1700 4300
+P 1750 4300
+F 0 "#PWR09" H 1750 4050 50  0001 C CNN
+F 1 "GND" H 1755 4127 50  0000 C CNN
+F 2 "" H 1750 4300 50  0001 C CNN
+F 3 "" H 1750 4300 50  0001 C CNN
+	1    1750 4300
 	1    0    0    -1
 $EndComp
@@
 	9000 5550 9050 5550
 $Comp
-L Regulator_Linear:AZ1117R-ADJ U1
+L Regulator_Linear:AMS1117 U1
 U 1 1 605CD92F
 P 1150 3900
-F 0 "U1" H 1150 4142 50  0000 C CNN
-F 1 "AZ1117R-ADJ" H 1150 4051 50  0000 C CNN
-F 2 "Package_TO_SOT_SMD:SOT-89-3" H 1150 4150 50  0001 C CIN
-F 3 "https://www.diodes.com/assets/Datasheets/products_inactive_data/AZ1117.pdf" H 1150 3900 50  0001 C CNN
+F 0 "U1" H 1150 4150 50  0000 C CNN
+F 1 "AMS1117-ADJ" H 1150 4050 50  0000 C CNN
+F 2 "Package_TO_SOT_SMD:SOT-223-3_TabPin2" H 1150 4150 50  0001 C CIN
+F 3 "" H 1150 3900 50  0001 C CNN
 	1    1150 3900
 	1    0    0    -1
@@
 L Device:R R2
 U 1 1 605FB724
-P 1500 4100
-F 0 "R2" H 1570 4146 50  0000 L CNN
-F 1 "1k" H 1570 4055 50  0000 L CNN
-F 2 "Resistor_SMD:R_0805_2012Metric_Pad1.20x1.40mm_HandSolder" V 1430 4100 50  0001 C CNN
-F 3 "~" H 1500 4100 50  0001 C CNN
-	1    1500 4100
+P 1550 4100
+F 0 "R2" H 1620 4146 50  0000 L CNN
+F 1 "1k" H 1620 4055 50  0000 L CNN
+F 2 "Resistor_SMD:R_0805_2012Metric_Pad1.20x1.40mm_HandSolder" V 1480 4100 50  0001 C CNN
+F 3 "~" H 1550 4100 50  0001 C CNN
+	1    1550 4100
 	-1   0    0    1
 $EndComp
 Wire Wire Line
-	1500 3950 1500 3900
-Wire Wire Line
-	1500 3900 1450 3900
-Wire Wire Line
-	1500 3900 1700 3900
-Connection ~ 1500 3900
-Wire Wire Line
-	1500 4250 1500 4300
-Wire Wire Line
-	1500 4300 1150 4300
+	1550 3950 1550 3900
+Wire Wire Line
+	1550 3900 1450 3900
+Wire Wire Line
+	1550 3900 1750 3900
+Connection ~ 1550 3900
+Wire Wire Line
+	1550 4250 1550 4300
+Wire Wire Line
+	1550 4300 1150 4300
 Wire Wire Line
 	1150 4300 1150 4200
@@
 L power:+4V #PWR08
 U 1 1 6066F638
-P 1700 3850
-F 0 "#PWR08" H 1700 3700 50  0001 C CNN
-F 1 "+4V" H 1715 4023 50  0000 C CNN
-F 2 "" H 1700 3850 50  0001 C CNN
-F 3 "" H 1700 3850 50  0001 C CNN
-	1    1700 3850
+P 1750 3850
+F 0 "#PWR08" H 1750 3700 50  0001 C CNN
+F 1 "+4V" H 1765 4023 50  0000 C CNN
+F 2 "" H 1750 3850 50  0001 C CNN
+F 3 "" H 1750 3850 50  0001 C CNN
+	1    1750 3850
 	1    0    0    -1
 $EndComp
@@
 F 0 "SW1" H 10450 4850 50  0000 C CNN
 F 1 "SW_Push" H 10450 4950 50  0000 C CNN
-F 2 "Button_Switch_SMD:SW_Push_1P1T_NO_CK_KMR2" H 10450 5250 50  0001 C CNN
+F 2 "Button_Switch_THT:SW_PUSH_6mm" H 10450 5250 50  0001 C CNN
 F 3 "~" H 10450 5250 50  0001 C CNN
 	1    10450 5050
