File: shield/GBAHD_Shield.kicad_pcb (KiCad board)
At the start: 2 copper layers, 53.4 x 53.1 mm, 38 parts, among them J1 Conn_01x01, J10 Conn_01x10, J11 Conn_02x03_Odd_Even, J12 Conn_01x01, J2 FFC_OGBA_32, J3 FFC_GBA-SP, J4 Conn_01x16, J5 FFC_OGBA_40, J6 Conn_01x06, J7 Conn_01x08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

Commit message: Switched Voltage Regulator to SOT-223 package and Push Button to THT
Parts:
- C1: moved to B.Cu
- SW1: footprint Button_Switch_SMD:SW_Push_1P1T_NO_CK_KMR2 -> Button_Switch_THT:SW_PUSH_6mm
- U1: value AZ1117R-ADJ -> AMS1117-ADJ; footprint Package_TO_SOT_SMD:SOT-89-3 -> Package_TO_SOT_SMD:SOT-223-3_TabPin2
- moved R2 5.17 mm to (73.8, 34.0)
- moved SW1 4.23 mm to (83.6, 38.6)
- moved C1 4.10 mm to (69.2, 39.8), turned to 180 degrees
- moved U1 1.96 mm to (68.6, 40.1)
- moved R1 1.37 mm to (74.0, 37.6)
- moved T1 0.80 mm to (86.7, 41.3)
- moved T2 0.80 mm to (86.7, 39.0)
- moved T3 0.80 mm to (86.7, 36.7)
- moved T4 0.80 mm to (86.7, 34.4)
- renumbered GND to GND1, VCC to VCC1
Connections:
- J10 pad 10: (no net) -> SP_ARSCL
- J10 pad 5: (no net) -> SP_ARD12
- J10 pad 8: (no net) -> Net-(J10-Pad8)
- J10 pad 9: (no net) -> SP_ARSDA
- J2 pad 1: (no net) -> Net-(J2-Pad1)
- J2 pad 23: (no net) -> Net-(J2-Pad23)
- J2 pad 24: (no net) -> Net-(J2-Pad24)
- J2 pad 26: (no net) -> Net-(J2-Pad26)
- J2 pad 27: (no net) -> Net-(J2-Pad27)
- J2 pad 28: (no net) -> Net-(J2-Pad28)
- J2 pad 29: (no net) -> Net-(J2-Pad29)
- J2 pad 3: (no net) -> Net-(J2-Pad3)
- J2 pad 30: (no net) -> Net-(J2-Pad30)
- J2 pad 31: (no net) -> Net-(J2-Pad31)
- J2 pad 32: (no net) -> Net-(J2-Pad32)
- J2 pad 4: (no net) -> Net-(J2-Pad4)
- J2 pad 5: (no net) -> Net-(J2-Pad5)
- J2 pad 6: (no net) -> Net-(J2-Pad6)
- J3 pad 1: (no net) -> Net-(J3-Pad1)
- J3 pad 23: (no net) -> Net-(J3-Pad23)
- J3 pad 24: (no net) -> Net-(J3-Pad24)
- J3 pad 26: (no net) -> Net-(J3-Pad26)
- J3 pad 27: (no net) -> Net-(J3-Pad27)
- J3 pad 28: (no net) -> Net-(J3-Pad28)
- J3 pad 29: (no net) -> Net-(J3-Pad29)
- J3 pad 3: (no net) -> Net-(J3-Pad3)
- J3 pad 30: (no net) -> Net-(J3-Pad30)
- J3 pad 31: (no net) -> Net-(J3-Pad31)
- J3 pad 33: (no net) -> Net-(J3-Pad33)
- J3 pad 34: (no net) -> Net-(J3-Pad34)
- J3 pad 4: (no net) -> Net-(J3-Pad4)
- J3 pad 5: (no net) -> Net-(J3-Pad5)
- J5 pad 1: (no net) -> Net-(J5-Pad1)
- J5 pad 2: (no net) -> Net-(J5-Pad2)
- J5 pad 24: (no net) -> Net-(J5-Pad24)
- J5 pad 25: (no net) -> Net-(J5-Pad25)
- J5 pad 27: (no net) -> Net-(J5-Pad27)
- J5 pad 28: (no net) -> Net-(J5-Pad28)
- J5 pad 29: (no net) -> Net-(J5-Pad29)
- J5 pad 30: (no net) -> Net-(J5-Pad30)
- J5 pad 31: (no net) -> Net-(J5-Pad31)
- J5 pad 32: (no net) -> Net-(J5-Pad32)
- J5 pad 33: (no net) -> Net-(J5-Pad33)
- J5 pad 34: (no net) -> Net-(J5-Pad34)
- J5 pad 36: (no net) -> Net-(J5-Pad36)
- J5 pad 37: (no net) -> Net-(J5-Pad37)
- J5 pad 38: (no net) -> Net-(J5-Pad38)
- J5 pad 39: (no net) -> Net-(J5-Pad39)
- J5 pad 4: (no net) -> Net-(J5-Pad4)
- J5 pad 40: (no net) -> Net-(J5-Pad40)
- J5 pad 5: (no net) -> Net-(J5-Pad5)
- J5 pad 7: (no net) -> Net-(J5-Pad7)
- J6 pad 1: (no net) -> AR_A0
- J6 pad 2: (no net) -> AR_A1
- J6 pad 3: (no net) -> AR_A2
- J6 pad 4: (no net) -> AR_A3
- J6 pad 5: (no net) -> AR_A4
- J6 pad 6: (no net) -> AR_A5
- J7 pad 1: (no net) -> SP_VIN
- J7 pad 6: (no net) -> SP_ARRES
- J7 pad 7: (no net) -> Net-(J7-Pad7)
- J7 pad 8: (no net) -> Net-(J7-Pad8)
- U3 pad 2: (no net) -> Net-(U3-Pad2)
- U3 pad 3: (no net) -> Net-(U3-Pad3)
- U3 pad 4: (no net) -> Net-(U3-Pad4)
- U3 pad 5: (no net) -> Net-(U3-Pad5)
- U3 pad 6: (no net) -> Net-(U3-Pad6)
- U3 pad 7: (no net) -> Net-(U3-Pad7)
- U3 pad 9: (no net) -> Net-(U3-Pad9)
- U5 pad 19: (no net) -> Net-(U5-Pad19)
- U5 pad 2: (no net) -> Net-(U5-Pad2)
- U5 pad 22: (no net) -> Net-(U5-Pad22)
- U5 pad 23: (no net) -> Net-(U5-Pad23)
- U5 pad 28: (no net) -> Net-(U5-Pad28)
- U5 pad 7: (no net) -> Net-(U5-Pad7)
- U5 pad 8: (no net) -> Net-(U5-Pad8)
Routing:
- net AT_RST: track 36.1 -> 45.5 mm, vias 1 -> 2
- net +4V: track 17.1 -> 25.2 mm
- net +5V: track 42.4 -> 45.2 mm
- net GB_SPS: track 48.3 -> 46.2 mm
- net Net-(R1-Pad2): track 4.26 -> 6.20 mm
- net GB_B1: track 47.2 -> 45.6 mm
- net +3V3: track 124.0 -> 125.5 mm
- net Net-(T4-Pad1): track 13.2 -> 11.8 mm
- net Net-(T1-Pad1): track 7.56 -> 6.48 mm
- net Net-(T3-Pad1): track 10.2 -> 9.32 mm
- net Net-(T2-Pad1): track 7.53 -> 6.89 mm
- net PIXEL_GRID: track 21.6 -> 22.2 mm, vias 0 -> 2
- net GND: vias 53 -> 57
Other:
- board text added: "ManCloud / hagi 2021 Designed in Germany v20210416_1"
- board text removed: "ManCloud 2021 Designed in Germany v20210416"

Commit message: Cleanup for shield pcb
Routing:
- net ~GBA_BUTTONS_EN~: track 25.0 -> 19.3 mm
- net SNS_LATCH: track 29.7 -> 33.1 mm
- net ICSP_MOSI: track 28.6 -> 25.3 mm
- net VCC: track 57.9 -> 60.0 mm
- net GBA_START: track 11.2 -> 13.2 mm
- net GBA_POWER_SEL: track 38.6 -> 39.2 mm
- net GND: vias 57 -> 58
